Commit message: changed naming scheme for back legs

File: quadruped_description/urdf/quadruped.urdf (robot description, URDF)
Before this commit: robot quadruped, 20 links, 19 joints
Links:
- removed link coxa_rl
- removed link coxa_rr
- removed link femur_rl
- removed link femur_rr
- removed link foot_rl
- removed link foot_rr
- removed link tibia_rl
- removed link tibia_rr
- added link coxa_bl, mass 0.63; visual mesh filename=package://quadruped_description/meshes/coxa.dae
- added link coxa_br, mass 0.63; visual mesh filename=package://quadruped_description/meshes/coxa.dae
- added link femur_bl, mass 0.481; visual mesh filename=package://quadruped_description/meshes/femur.dae
- added link femur_br, mass 0.481; visual mesh filename=package://quadruped_description/meshes/femur.dae
- added link foot_bl
- added link foot_br
- added link tibia_bl, mass 0.29; collision mesh filename=package://quadruped_description/meshes/tibia.dae; visual mesh filename=package://quadruped_description/meshes/tibia.dae
- added link tibia_br, mass 0.29; collision mesh filename=package://quadruped_description/meshes/tibia.dae; visual mesh filename=package://quadruped_description/meshes/tibia.dae
Joints:
- removed joint joint_ankle_rl
- removed joint joint_ankle_rr
- removed joint joint_foot_rl
- removed joint joint_foot_rr
- removed joint joint_hip_rl
- removed joint joint_hip_rr
- removed joint joint_knee_rl
- removed joint joint_knee_rr
- added joint joint_ankle_bl: type revolute, parent femur_bl, child tibia_bl, origin xyz=0.2032 0 0 rpy=0 0 0 , axis 0 0 1, limit lower=-3 upper=3 effort=30.0 velocity=6
- added joint joint_ankle_br: type revolute, parent femur_br, child tibia_br, origin xyz=0.2032 0 0 rpy=0 0 0 , axis 0 0 1, limit lower=-3 upper=3 effort=30.0 velocity=6
- added joint joint_foot_bl: type fixed, parent tibia_bl, child foot_bl, origin xyz=0.2032 0 0 rpy=0 0 0 
- added joint joint_foot_br: type fixed, parent tibia_br, child foot_br, origin xyz=0.2032 0 0 rpy=0 0 0 
- added joint joint_hip_bl: type revolute, parent body, child coxa_bl, origin xyz=-0.1016 -0.1524 0 rpy=1.57 0 -1.57, axis 0 0 1, limit lower=-3 upper=3 effort=30.0 velocity=6
- added joint joint_hip_br: type revolute, parent body, child coxa_br, origin xyz=-0.1016 0.1524 0 rpy=1.57 0 -1.57, axis 0 0 1, limit lower=-3 upper=3 effort=30.0 velocity=6
- added joint joint_knee_bl: type revolute, parent coxa_bl, child femur_bl, origin xyz=0 0 0.0762 rpy=1.57 0 -1.57, axis 0 0 1, limit lower=-3 upper=3 effort=30.0 velocity=6
- added joint joint_knee_br: type revolute, parent coxa_br, child femur_br, origin xyz=0 0 0.0762 rpy=1.57 0 -1.57, axis 0 0 1, limit lower=-3 upper=3 effort=30.0 velocity=6

Commit message: fixed right left mixup

File: quadruped_description/urdf/quadruped.urdf (robot description, URDF)
Before this commit: robot quadruped, 20 links, 19 joints
Joints:
- joint joint_foot_fr: parent femur_fr -> tibia_fr
- joint joint_hip_bl: origin xyz=-0.1016 -0.1524 0 rpy=1.57 0 -1.57 -> xyz=-0.1016 0.1524 0 rpy=1.57 0 -1.57
- joint joint_hip_br: origin xyz=-0.1016 0.1524 0 rpy=1.57 0 -1.57 -> xyz=-0.1016 -0.1524 0 rpy=1.57 0 -1.57
- joint joint_hip_fl: origin xyz=0.1778 -0.1524 0 rpy=1.57 0 -1.57 -> xyz=0.1778 0.1524 0 rpy=1.57 0 -1.57
- joint joint_hip_fr: origin xyz=0.1778 0.1524 0 rpy=1.57 0 -1.57 -> xyz=0.1778 -0.1524 0 rpy=1.57 0 -1.57

Commit message: implemented stability measurements

File: quadruped_description/urdf/quadruped.urdf (robot description, URDF)
Before this commit: robot quadruped, 20 links, 19 joints
Links:
- link foot_br: mass None -> 0.0001; geometry visual sphere radius=0.001
- link foot_fl: mass None -> 0.29

Commit message: Added tail controller, updated gail controller

File: quadruped_description/urdf/quadruped.urdf (robot description, URDF)
Before this commit: robot quadruped, 20 links, 19 joints
Links:
- added link body_com, mass 0.0001
- added link coxa_bl_com, mass 0.0001
- added link coxa_br_com, mass 0.0001
- added link coxa_fl_com, mass 0.0001
- added link coxa_fr_com, mass 0.0001
- added link femur_bl_com, mass 0.0001
- added link femur_br_com, mass 0.0001
- added link femur_fl_com, mass 0.0001
- added link femur_fr_com, mass 0.0001
- added link tail_com, mass 0.0001
- added link tailbase_com, mass 0.0001
- added link tibia_bl_com, mass 0.0001
- added link tibia_br_com, mass 0.0001
- added link tibia_fl_com, mass 0.0001
- added link tibia_fr_com, mass 0.0001
- link foot_bl: mass None -> 0.0001
- link foot_br: mass None -> 0.0001
- link foot_fl: mass None -> 0.0001
- link foot_fr: mass None -> 0.0001
Joints:
- added joint joint_body_com: type fixed, parent body, child body_com, origin xyz=0.01781 0.0 0.00882 rpy=0 0 0 
- added joint joint_coxa_bl_com: type fixed, parent coxa_bl, child coxa_bl_com, origin xyz=0.0 0.0 0.04183 rpy=0 0 0 
- added joint joint_coxa_br_com: type fixed, parent coxa_br, child coxa_br_com, origin xyz=0.0 0.0 0.04183 rpy=0 0 0 
- added joint joint_coxa_fl_com: type fixed, parent coxa_fl, child coxa_fl_com, origin xyz=0.0 0.0 0.04183 rpy=0 0 0 
- added joint joint_coxa_fr_com: type fixed, parent coxa_fr, child coxa_fr_com, origin xyz=0.0 0.0 0.04183 rpy=0 0 0 
- added joint joint_femur_bl_com: type fixed, parent femur_bl, child femur_bl_com, origin xyz=0.08660 0.0 0.0 rpy=0 0 0 
- added joint joint_femur_br_com: type fixed, parent femur_br, child femur_br_com, origin xyz=0.08660 0.0 0.0 rpy=0 0 0 
- added joint joint_femur_fl_com: type fixed, parent femur_fl, child femur_fl_com, origin xyz=0.08660 0.0 0.0 rpy=0 0 0 
- added joint joint_femur_fr_com: type fixed, parent femur_fr, child femur_fr_com, origin xyz=0.08660 0.0 0.0 rpy=0 0 0 
- added joint joint_tail_com: type fixed, parent tail, child tail_com, origin xyz=0.15694 0.0 0.0 rpy=0 0 0 
- added joint joint_tailbase_com: type fixed, parent tailbase, child tailbase_com, origin xyz=0.0 0.0 0.04244 rpy=0 0 0 
- added joint joint_tibia_bl_com: type fixed, parent tibia_bl, child tibia_bl_com, origin xyz=0.10609 0.0 0.0 rpy=0 0 0 
- added joint joint_tibia_br_com: type fixed, parent tibia_br, child tibia_br_com, origin xyz=0.10609 0.0 0.0 rpy=0 0 0 
- added joint joint_tibia_fl_com: type fixed, parent tibia_fl, child tibia_fl_com, origin xyz=0.10609 0.0 0.0 rpy=0 0 0 
- added joint joint_tibia_fr_com: type fixed, parent tibia_fr, child tibia_fr_com, origin xyz=0.10609 0.0 0.0 rpy=0 0 0 

Commit message: implemented stability controller

File: quadruped_description/urdf/quadruped.urdf (robot description, URDF)
Before this commit: robot quadruped, 20 links, 19 joints
Links:
- link foot_br: mass 0.0001 -> None; geometry 
- link foot_fl: mass 0.29 -> None
